File: hw/rotary_encoder_board.brd (EAGLE design)
At the start: 35 x 30 mm, 2 parts, among them SW1 EC12E_SW

Commit message: use angled pinheaders
Parts:
- removed ENCODER: (no value), con-lstb:MA04-1
- added JP1: (no value), pinhead:1X04/90
Connections:
- net ENCODER_A: now also JP1.2; no longer ENCODER.3
- net ENCODER_B: now also JP1.1; no longer ENCODER.4
- net ENCODER_BTN: now also JP1.3; no longer ENCODER.2
- net GND: now also JP1.4; no longer ENCODER.1
Changed lines of the file:
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@@
 </autorouter>
 <elements>
-<element name="ENCODER" library="con-lstb" package="MA04-1" value="" x="27.94" y="15.24" rot="MR270">
-<attribute name="OC_NEWARK" value="unknown" x="27.94" y="15.24" size="1.778" layer="28" rot="MR270" display="off"/>
-<attribute name="MPN" value="" x="27.94" y="15.24" size="1.778" layer="28" rot="MR270" display="off"/>
-<attribute name="MF" value="" x="27.94" y="15.24" size="1.778" layer="28" rot="MR270" display="off"/>
-<attribute name="OC_FARNELL" value="unknown" x="27.94" y="15.24" size="1.778" layer="28" rot="MR270" display="off"/>
-</element>
 <element name="SW1" library="switch-alps" package="ALPS_EC12E_SW" value="EC12E_SW" x="15.24" y="15.24">
 <attribute name="OC_NEWARK" value="74M1068" x="15.24" y="15.24" size="1.778" layer="27" display="off"/>
@@
 <attribute name="OC_FARNELL" value="1520813" x="15.24" y="15.24" size="1.778" layer="27" display="off"/>
 </element>
+<element name="JP1" library="pinhead" package="1X04/90" value="" x="31.75" y="15.24" rot="MR90"/>
 </elements>
 <signals>
 <signal name="GND">
-<contactref element="ENCODER" pad="1"/>
 <contactref element="SW1" pad="C"/>
 <contactref element="SW1" pad="D"/>
@@
 <vertex x="-1.27" y="-1.27"/>
 </polygon>
+<contactref element="JP1" pad="4"/>
 </signal>
 <signal name="ENCODER_BTN">
-<contactref element="ENCODER" pad="2"/>
 <contactref element="SW1" pad="E"/>
 <wire x1="17.74" y1="22.24" x2="17.74" y2="22.82" width="0.4064" layer="1"/>
@@
 <wire x1="31.75" y1="21.59" x2="31.75" y2="17.78" width="0.4064" layer="1"/>
 <wire x1="31.75" y1="17.78" x2="30.48" y2="16.51" width="0.4064" layer="1"/>
-<wire x1="30.48" y1="16.51" x2="27.94" y2="16.51" width="0.4064" layer="1"/>
+<contactref element="JP1" pad="3"/>
+<wire x1="27.94" y1="16.51" x2="30.48" y2="16.51" width="0.4064" layer="1"/>
 </signal>
 <signal name="ENCODER_A">
-<contactref element="ENCODER" pad="3"/>
 <contactref element="SW1" pad="A"/>
 <wire x1="12.74" y1="7.74" x2="12.74" y2="6.31" width="0.4064" layer="1"/>
@@
 <wire x1="31.75" y1="8.89" x2="31.75" y2="12.7" width="0.4064" layer="1"/>
 <wire x1="31.75" y1="12.7" x2="30.48" y2="13.97" width="0.4064" layer="1"/>
-<wire x1="30.48" y1="13.97" x2="27.94" y2="13.97" width="0.4064" layer="1"/>
+<contactref element="JP1" pad="2"/>
+<wire x1="27.94" y1="13.97" x2="30.48" y2="13.97" width="0.4064" layer="1"/>
 </signal>
 <signal name="ENCODER_B">
-<contactref element="ENCODER" pad="4"/>
 <contactref element="SW1" pad="B"/>
 <wire x1="17.74" y1="7.74" x2="17.74" y2="7.66" width="0.4064" layer="1"/>
@@
 <wire x1="19.05" y1="6.35" x2="24.13" y2="6.35" width="0.4064" layer="1"/>
 <wire x1="24.13" y1="6.35" x2="27.94" y2="10.16" width="0.4064" layer="1"/>
-<wire x1="27.94" y1="10.16" x2="27.94" y2="11.43" width="0.4064" layer="1"/>
+<contactref element="JP1" pad="1"/>
+<wire x1="27.94" y1="11.43" x2="27.94" y2="10.16" width="0.4064" layer="1"/>
 </signal>
 </signals>
