File: hw/rotary_encoder_board.sch (EAGLE design)
At the start: 2 parts, among them SW1 EC12E_SW

Commit message: use angled pinheaders
Parts:
- removed ENCODER: (no value), con-lstb:MA04-1
- added JP1: (no value), pinhead:PINHD-1X4/90
Connections:
- net ENCODER_A: now also JP1.2; no longer ENCODER.3
- net ENCODER_B: now also JP1.1; no longer ENCODER.4
- net ENCODER_BTN: now also JP1.3; no longer ENCODER.2
- net GND: now also JP1.4; no longer ENCODER.1
Changed lines of the file:
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@@
 </classes>
 <parts>
-<part name="ENCODER" library="con-lstb" deviceset="MA04-1" device=""/>
 <part name="GND1" library="supply1" deviceset="GND" device=""/>
 <part name="SW1" library="switch-alps" deviceset="EC12E_SW" device=""/>
 <part name="GND2" library="supply1" deviceset="GND" device=""/>
 <part name="GND3" library="supply1" deviceset="GND" device=""/>
+<part name="JP1" library="pinhead" deviceset="PINHD-1X4" device="/90"/>
 </parts>
 <sheets>
@@
 </plain>
 <instances>
-<instance part="ENCODER" gate="1" x="33.02" y="7.62" rot="R180"/>
-<instance part="GND1" gate="1" x="22.86" y="12.7" rot="R270"/>
+<instance part="GND1" gate="1" x="20.32" y="12.7" rot="R270"/>
 <instance part="SW1" gate="G$1" x="55.88" y="7.62"/>
 <instance part="SW1" gate="G$2" x="76.2" y="10.16" rot="MR270"/>
 <instance part="GND2" gate="1" x="55.88" y="2.54"/>
 <instance part="GND3" gate="1" x="76.2" y="2.54"/>
+<instance part="JP1" gate="A" x="30.48" y="10.16" rot="MR180"/>
 </instances>
 <busses>
@@
 <nets>
 <net name="GND" class="0">
-<segment>
-<pinref part="ENCODER" gate="1" pin="1"/>
-<pinref part="GND1" gate="1" pin="GND"/>
-</segment>
 <segment>
 <pinref part="SW1" gate="G$1" pin="C"/>
@@
 <pinref part="GND3" gate="1" pin="GND"/>
 </segment>
+<segment>
+<pinref part="GND1" gate="1" pin="GND"/>
+<pinref part="JP1" gate="A" pin="4"/>
+<wire x1="27.94" y1="12.7" x2="22.86" y2="12.7" width="0.1524" layer="91"/>
+</segment>
 </net>
 <net name="ENCODER_BTN" class="0">
 <segment>
-<pinref part="ENCODER" gate="1" pin="2"/>
-<wire x1="25.4" y1="10.16" x2="17.78" y2="10.16" width="0.1524" layer="91"/>
+<wire x1="27.94" y1="10.16" x2="17.78" y2="10.16" width="0.1524" layer="91"/>
 <label x="17.78" y="10.16" size="1.27" layer="95" rot="R180" xref="yes"/>
+<pinref part="JP1" gate="A" pin="3"/>
 </segment>
 <segment>
@@
 <net name="ENCODER_A" class="0">
 <segment>
-<pinref part="ENCODER" gate="1" pin="3"/>
-<wire x1="17.78" y1="7.62" x2="25.4" y2="7.62" width="0.1524" layer="91"/>
+<wire x1="17.78" y1="7.62" x2="27.94" y2="7.62" width="0.1524" layer="91"/>
 <label x="17.78" y="7.62" size="1.27" layer="95" rot="R180" xref="yes"/>
+<pinref part="JP1" gate="A" pin="2"/>
 </segment>
 <segment>
@@
 <net name="ENCODER_B" class="0">
 <segment>
-<pinref part="ENCODER" gate="1" pin="4"/>
-<wire x1="25.4" y1="5.08" x2="17.78" y2="5.08" width="0.1524" layer="91"/>
+<wire x1="27.94" y1="5.08" x2="17.78" y2="5.08" width="0.1524" layer="91"/>
 <label x="17.78" y="5.08" size="1.27" layer="95" rot="R180" xref="yes"/>
+<pinref part="JP1" gate="A" pin="1"/>
 </segment>
 <segment>
