File: hw/bbb_connection_board.sch (EAGLE design)
At the start: 2 parts, among them P8 MA23-2

Commit message: schematic of bbb connection board
Parts:
- added ENCODER, PWR_BTN_LED: (no value), con-lstb:MA04-1
- added R1, R2, R3, R4, R5: 10k, rcl:R-EU_R0805
- added R6: 330R, rcl:R-EU_R0805
- added T1: (no value), transistor:BC847A-NPN-SOT23-BEC
- renumbered JP1 to POWER_SUPPLY
Connections:
- removed net ENCODER_TASTER: P8.8
- removed net PWR_TASTER: P8.7
- new net ENCODER_BTN: ENCODER.2, P8.8, R2.1
- new net LED_OUT: PWR_BTN_LED.4, R6.2
- new net N$1: R5.2, T1.B
- new net N$3: R6.1, T1.C
- new net PWR_BTN: P8.7, PWR_BTN_LED.2, R1.1
- net +3V3: now also PWR_BTN_LED.3, R1.2, R2.2, R3.2, R4.2
- net ENCODER_A: now also ENCODER.3, R3.1
- net ENCODER_B: now also ENCODER.4, R4.1
- net GND: now also ENCODER.1, PWR_BTN_LED.1, T1.E
- net PWR_LED: now also R5.1
Changed lines of the file:
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@@
 <parts>
 <part name="P8" library="con-lstb-mod" deviceset="MA23-2" device=""/>
-<part name="JP1" library="jumper" deviceset="JP1E" device=""/>
+<part name="POWER_SUPPLY" library="jumper" deviceset="JP1E" device=""/>
 <part name="GND1" library="supply1" deviceset="GND" device=""/>
 <part name="GND2" library="supply1" deviceset="GND" device=""/>
 <part name="GND3" library="supply1" deviceset="GND" device=""/>
 <part name="+3V1" library="supply1" deviceset="+3V3" device=""/>
+<part name="R1" library="rcl" deviceset="R-EU_" device="R0805" value="10k"/>
+<part name="R2" library="rcl" deviceset="R-EU_" device="R0805" value="10k"/>
+<part name="R3" library="rcl" deviceset="R-EU_" device="R0805" value="10k"/>
+<part name="R4" library="rcl" deviceset="R-EU_" device="R0805" value="10k"/>
+<part name="+3V2" library="supply1" deviceset="+3V3" device=""/>
+<part name="+3V3" library="supply1" deviceset="+3V3" device=""/>
+<part name="+3V4" library="supply1" deviceset="+3V3" device=""/>
+<part name="+3V5" library="supply1" deviceset="+3V3" device=""/>
+<part name="ENCODER" library="con-lstb" deviceset="MA04-1" device=""/>
+<part name="PWR_BTN_LED" library="con-lstb" deviceset="MA04-1" device=""/>
+<part name="GND4" library="supply1" deviceset="GND" device=""/>
+<part name="GND5" library="supply1" deviceset="GND" device=""/>
+<part name="+3V6" library="supply1" deviceset="+3V3" device=""/>
+<part name="T1" library="transistor" deviceset="*-NPN-" device="SOT23-BEC" technology="BC847A"/>
+<part name="GND6" library="supply1" deviceset="GND" device=""/>
+<part name="R5" library="rcl" deviceset="R-EU_" device="R0805" value="10k"/>
+<part name="R6" library="rcl" deviceset="R-EU_" device="R0805" value="330R"/>
 </parts>
 <sheets>
@@
 <instances>
 <instance part="P8" gate="G$1" x="40.64" y="68.58" rot="R180"/>
-<instance part="JP1" gate="A" x="30.48" y="83.82" rot="MR270"/>
+<instance part="POWER_SUPPLY" gate="A" x="30.48" y="83.82" rot="MR270"/>
 <instance part="GND1" gate="1" x="25.4" y="66.04" rot="R270"/>
 <instance part="GND2" gate="1" x="45.72" y="66.04" rot="R90"/>
 <instance part="GND3" gate="1" x="35.56" y="83.82" rot="R90"/>
 <instance part="+3V1" gate="G$1" x="35.56" y="81.28" rot="MR90"/>
+<instance part="R1" gate="G$1" x="83.82" y="35.56"/>
+<instance part="R2" gate="G$1" x="83.82" y="27.94"/>
+<instance part="R3" gate="G$1" x="83.82" y="20.32"/>
+<instance part="R4" gate="G$1" x="83.82" y="12.7"/>
+<instance part="+3V2" gate="G$1" x="91.44" y="35.56" rot="MR90"/>
+<instance part="+3V3" gate="G$1" x="91.44" y="27.94" rot="MR90"/>
+<instance part="+3V4" gate="G$1" x="91.44" y="20.32" rot="MR90"/>
+<instance part="+3V5" gate="G$1" x="91.44" y="12.7" rot="MR90"/>
+<instance part="ENCODER" gate="1" x="109.22" y="73.66" rot="R180"/>
+<instance part="PWR_BTN_LED" gate="1" x="109.22" y="53.34" rot="R180"/>
+<instance part="GND4" gate="1" x="99.06" y="78.74" rot="R270"/>
+<instance part="GND5" gate="1" x="99.06" y="58.42" rot="R270"/>
+<instance part="+3V6" gate="G$1" x="96.52" y="53.34" rot="MR270"/>
+<instance part="T1" gate="G$1" x="127" y="20.32"/>
+<instance part="GND6" gate="1" x="129.54" y="12.7"/>
+<instance part="R5" gate="G$1" x="119.38" y="20.32"/>
+<instance part="R6" gate="G$1" x="129.54" y="30.48" rot="R90"/>
 </instances>
 <busses>
@@
 </segment>
 <segment>
-<pinref part="JP1" gate="A" pin="1"/>
+<pinref part="POWER_SUPPLY" gate="A" pin="1"/>
 <pinref part="GND3" gate="1" pin="GND"/>
 </segment>
+<segment>
+<pinref part="ENCODER" gate="1" pin="1"/>
+<pinref part="GND4" gate="1" pin="GND"/>
+</segment>
+<segment>
+<pinref part="PWR_BTN_LED" gate="1" pin="1"/>
+<pinref part="GND5" gate="1" pin="GND"/>
+</segment>
+<segment>
+<pinref part="T1" gate="G$1" pin="E"/>
+<pinref part="GND6" gate="1" pin="GND"/>
+</segment>
 </net>
 <net name="+3V3" class="0">
 <segment>
-<pinref part="JP1" gate="A" pin="2"/>
+<pinref part="POWER_SUPPLY" gate="A" pin="2"/>
 <pinref part="+3V1" gate="G$1" pin="+3V3"/>
+</segment>
+<segment>
+<pinref part="R1" gate="G$1" pin="2"/>
+<pinref part="+3V2" gate="G$1" pin="+3V3"/>
+</segment>
+<segment>
+<pinref part="R2" gate="G$1" pin="2"/>
+<pinref part="+3V3" gate="G$1" pin="+3V3"/>
+</segment>
+<segment>
+<pinref part="R3" gate="G$1" pin="2"/>
+<pinref part="+3V4" gate="G$1" pin="+3V3"/>
+</segment>
+<segment>
+<pinref part="R4" gate="G$1" pin="2"/>
+<pinref part="+3V5" gate="G$1" pin="+3V3"/>
+</segment>
+<segment>
+<pinref part="PWR_BTN_LED" gate="1" pin="3"/>
+<pinref part="+3V6" gate="G$1" pin="+3V3"/>
+<wire x1="99.06" y1="53.34" x2="101.6" y2="53.34" width="0.1524" layer="91"/>
 </segment>
 </net>
@@
 <label x="20.32" y="43.18" size="1.27" layer="95" rot="R180" xref="yes"/>
 </segment>
+<segment>
+<pinref part="R5" gate="G$1" pin="1"/>
+<wire x1="114.3" y1="20.32" x2="111.76" y2="20.32" width="0.1524" layer="91"/>
+<label x="111.76" y="20.32" size="1.27" layer="95" rot="R180" xref="yes"/>
+</segment>
 </net>
 <net name="ENCODER_B" class="0">
@@
 <label x="20.32" y="53.34" size="1.27" layer="95" rot="R180" xref="yes"/>
 </segment>
+<segment>
+<pinref part="R4" gate="G$1" pin="1"/>
+<wire x1="71.12" y1="12.7" x2="78.74" y2="12.7" width="0.1524" layer="91"/>
+<label x="71.12" y="12.7" size="1.27" layer="95" rot="R180" xref="yes"/>
+</segment>
+<segment>
+<pinref part="ENCODER" gate="1" pin="4"/>
+<wire x1="101.6" y1="71.12" x2="93.98" y2="71.12" width="0.1524" layer="91"/>
+<label x="93.98" y="71.12" size="1.27" layer="95" rot="R180" xref="yes"/>
+</segment>
 </net>
 <net name="ENCODER_A" class="0">
@@
 <label x="50.8" y="53.34" size="1.27" layer="95" xref="yes"/>
 </segment>
-</net>
-<net name="PWR_TASTER" class="0">
+<segment>
+<pinref part="R3" gate="G$1" pin="1"/>
+<wire x1="71.12" y1="20.32" x2="78.74" y2="20.32" width="0.1524" layer="91"/>
+<label x="71.12" y="20.32" size="1.27" layer="95" rot="R180" xref="yes"/>
+</segment>
+<segment>
+<pinref part="ENCODER" gate="1" pin="3"/>
+<wire x1="101.6" y1="73.66" x2="93.98" y2="73.66" width="0.1524" layer="91"/>
+<label x="93.98" y="73.66" size="1.27" layer="95" rot="R180" xref="yes"/>
+</segment>
+</net>
+<net name="PWR_BTN" class="0">
 <segment>
 <pinref part="P8" gate="G$1" pin="7"/>
@@
 <label x="20.32" y="58.42" size="1.27" layer="95" rot="R180" xref="yes"/>
 </segment>
-</net>
-<net name="ENCODER_TASTER" class="0">
+<segment>
+<pinref part="R1" gate="G$1" pin="1"/>
+<wire x1="78.74" y1="35.56" x2="71.12" y2="35.56" width="0.1524" layer="91"/>
+<label x="71.12" y="35.56" size="1.27" layer="95" rot="R180" xref="yes"/>
+</segment>
+<segment>
+<pinref part="PWR_BTN_LED" gate="1" pin="2"/>
+<wire x1="101.6" y1="55.88" x2="93.98" y2="55.88" width="0.1524" layer="91"/>
+<label x="93.98" y="55.88" size="1.27" layer="95" rot="R180" xref="yes"/>
+</segment>
+</net>
+<net name="ENCODER_BTN" class="0">
 <segment>
 <pinref part="P8" gate="G$1" pin="8"/>
@@
 <label x="50.8" y="58.42" size="1.27" layer="95" xref="yes"/>
 </segment>
-</net>
+<segment>
+<pinref part="R2" gate="G$1" pin="1"/>
+<wire x1="78.74" y1="27.94" x2="71.12" y2="27.94" width="0.1524" layer="91"/>
+<label x="71.12" y="27.94" size="1.27" layer="95" rot="R180" xref="yes"/>
+</segment>
+<segment>
+<pinref part="ENCODER" gate="1" pin="2"/>
+<wire x1="101.6" y1="76.2" x2="93.98" y2="76.2" width="0.1524" layer="91"/>
+<label x="93.98" y="76.2" size="1.27" layer="95" rot="R180" xref="yes"/>
+</segment>
+</net>
+<net name="N$1" class="0">
+<segment>
+<pinref part="T1" gate="G$1" pin="B"/>
+<pinref part="R5" gate="G$1" pin="2"/>
+</segment>
+</net>
+<net name="N$3" class="0">
+<segment>
+<pinref part="T1" gate="G$1" pin="C"/>
+<pinref part="R6" gate="G$1" pin="1"/>
+</segment>
+</net>
+<net name="LED_OUT" class="0">
+<segment>
+<pinref part="R6" gate="G$1" pin="2"/>
+<wire x1="129.54" y1="35.56" x2="129.54" y2="40.64" width="0.1524" layer="91"/>
+<label x="129.54" y="40.64" size="1.27" layer="95" rot="R90" xref="yes"/>
+</segment>
+<segment>
+<pinref part="PWR_BTN_LED" gate="1" pin="4"/>
+<wire x1="101.6" y1="50.8" x2="93.98" y2="50.8" width="0.1524" layer="91"/>
+<label x="93.98" y="50.8" size="1.27" layer="95" rot="R180" xref="yes"/>
+</segment>
+</net>

Commit message: bbb connection board routed
Parts:
- renumbered POWER_SUPPLY to PWR_IN
Changed lines of the file:
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@@
 <parts>
 <part name="P8" library="con-lstb-mod" deviceset="MA23-2" device=""/>
-<part name="POWER_SUPPLY" library="jumper" deviceset="JP1E" device=""/>
+<part name="PWR_IN" library="jumper" deviceset="JP1E" device=""/>
 <part name="GND1" library="supply1" deviceset="GND" device=""/>
 <part name="GND2" library="supply1" deviceset="GND" device=""/>
@@
 <instances>
 <instance part="P8" gate="G$1" x="40.64" y="68.58" rot="R180"/>
-<instance part="POWER_SUPPLY" gate="A" x="30.48" y="83.82" rot="MR270"/>
+<instance part="PWR_IN" gate="A" x="30.48" y="83.82" rot="MR270"/>
 <instance part="GND1" gate="1" x="25.4" y="66.04" rot="R270"/>
 <instance part="GND2" gate="1" x="45.72" y="66.04" rot="R90"/>
@@
 </segment>
 <segment>
-<pinref part="POWER_SUPPLY" gate="A" pin="1"/>
+<pinref part="PWR_IN" gate="A" pin="1"/>
 <pinref part="GND3" gate="1" pin="GND"/>
 </segment>
@@
 <net name="+3V3" class="0">
 <segment>
-<pinref part="POWER_SUPPLY" gate="A" pin="2"/>
+<pinref part="PWR_IN" gate="A" pin="2"/>
 <pinref part="+3V1" gate="G$1" pin="+3V3"/>
 </segment>

Commit message: use angled pinheaders
Parts:
- removed PWR_BTN_LED: (no value), con-lstb:MA04-1
- removed PWR_IN: (no value), jumper:JP1E
- added PWN_BTN_LED: (no value), pinhead:PINHD-1X4/90
- added PWR_CON: (no value), pinhead:PINHD-1X2/90
- ENCODER: device con-lstb:MA04-1 -> pinhead:PINHD-1X4/90
Connections:
- net +3V3: now also PWN_BTN_LED.2, PWR_CON.1; no longer PWR_BTN_LED.3, PWR_IN.2
- net ENCODER_A: now also ENCODER.2; no longer ENCODER.3
- net ENCODER_B: now also ENCODER.1; no longer ENCODER.4
- net ENCODER_BTN: now also ENCODER.3; no longer ENCODER.2
- net GND: now also ENCODER.4, PWN_BTN_LED.4, PWR_CON.2; no longer ENCODER.1, PWR_BTN_LED.1, PWR_IN.1
- net LED_OUT: now also PWN_BTN_LED.1; no longer PWR_BTN_LED.4
- net PWR_BTN: now also PWN_BTN_LED.3; no longer PWR_BTN_LED.2
Changed lines of the file:
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@@
 <parts>
 <part name="P8" library="con-lstb-mod" deviceset="MA23-2" device=""/>
-<part name="PWR_IN" library="jumper" deviceset="JP1E" device=""/>
 <part name="GND1" library="supply1" deviceset="GND" device=""/>
 <part name="GND2" library="supply1" deviceset="GND" device=""/>
@@
 <part name="+3V4" library="supply1" deviceset="+3V3" device=""/>
 <part name="+3V5" library="supply1" deviceset="+3V3" device=""/>
-<part name="ENCODER" library="con-lstb" deviceset="MA04-1" device=""/>
-<part name="PWR_BTN_LED" library="con-lstb" deviceset="MA04-1" device=""/>
 <part name="GND4" library="supply1" deviceset="GND" device=""/>
 <part name="GND5" library="supply1" deviceset="GND" device=""/>
@@
 <part name="R5" library="rcl" deviceset="R-EU_" device="R0805" value="10k"/>
 <part name="R6" library="rcl" deviceset="R-EU_" device="R0805" value="330R"/>
+<part name="PWR_CON" library="pinhead" deviceset="PINHD-1X2" device="/90"/>
+<part name="ENCODER" library="pinhead" deviceset="PINHD-1X4" device="/90"/>
+<part name="PWN_BTN_LED" library="pinhead" deviceset="PINHD-1X4" device="/90"/>
 </parts>
 <sheets>
@@
 <instances>
 <instance part="P8" gate="G$1" x="40.64" y="68.58" rot="R180"/>
-<instance part="PWR_IN" gate="A" x="30.48" y="83.82" rot="MR270"/>
 <instance part="GND1" gate="1" x="25.4" y="66.04" rot="R270"/>
 <instance part="GND2" gate="1" x="45.72" y="66.04" rot="R90"/>
-<instance part="GND3" gate="1" x="35.56" y="83.82" rot="R90"/>
-<instance part="+3V1" gate="G$1" x="35.56" y="81.28" rot="MR90"/>
+<instance part="GND3" gate="1" x="40.64" y="81.28" rot="R270"/>
+<instance part="+3V1" gate="G$1" x="40.64" y="83.82" rot="MR270"/>
 <instance part="R1" gate="G$1" x="83.82" y="35.56"/>
 <instance part="R2" gate="G$1" x="83.82" y="27.94"/>
@@
 <instance part="+3V4" gate="G$1" x="91.44" y="20.32" rot="MR90"/>
 <instance part="+3V5" gate="G$1" x="91.44" y="12.7" rot="MR90"/>
-<instance part="ENCODER" gate="1" x="109.22" y="73.66" rot="R180"/>
-<instance part="PWR_BTN_LED" gate="1" x="109.22" y="53.34" rot="R180"/>
-<instance part="GND4" gate="1" x="99.06" y="78.74" rot="R270"/>
-<instance part="GND5" gate="1" x="99.06" y="58.42" rot="R270"/>
-<instance part="+3V6" gate="G$1" x="96.52" y="53.34" rot="MR270"/>
+<instance part="GND4" gate="1" x="96.52" y="78.74" rot="R270"/>
+<instance part="GND5" gate="1" x="96.52" y="58.42" rot="R270"/>
+<instance part="+3V6" gate="G$1" x="96.52" y="53.34" rot="R90"/>
 <instance part="T1" gate="G$1" x="127" y="20.32"/>
 <instance part="GND6" gate="1" x="129.54" y="12.7"/>
 <instance part="R5" gate="G$1" x="119.38" y="20.32"/>
 <instance part="R6" gate="G$1" x="129.54" y="30.48" rot="R90"/>
+<instance part="PWR_CON" gate="G$1" x="53.34" y="81.28"/>
+<instance part="ENCODER" gate="A" x="106.68" y="76.2" rot="MR180"/>
+<instance part="PWN_BTN_LED" gate="A" x="106.68" y="55.88" rot="MR180"/>
 </instances>
 <busses>
@@
 </segment>
 <segment>
-<pinref part="PWR_IN" gate="A" pin="1"/>
-<pinref part="GND3" gate="1" pin="GND"/>
-</segment>
-<segment>
-<pinref part="ENCODER" gate="1" pin="1"/>
-<pinref part="GND4" gate="1" pin="GND"/>
-</segment>
-<segment>
-<pinref part="PWR_BTN_LED" gate="1" pin="1"/>
-<pinref part="GND5" gate="1" pin="GND"/>
-</segment>
-<segment>
 <pinref part="T1" gate="G$1" pin="E"/>
 <pinref part="GND6" gate="1" pin="GND"/>
 </segment>
+<segment>
+<pinref part="GND3" gate="1" pin="GND"/>
+<pinref part="PWR_CON" gate="G$1" pin="2"/>
+<wire x1="43.18" y1="81.28" x2="50.8" y2="81.28" width="0.1524" layer="91"/>
+</segment>
+<segment>
+<pinref part="GND4" gate="1" pin="GND"/>
+<pinref part="ENCODER" gate="A" pin="4"/>
+<wire x1="99.06" y1="78.74" x2="104.14" y2="78.74" width="0.1524" layer="91"/>
+</segment>
+<segment>
+<pinref part="GND5" gate="1" pin="GND"/>
+<pinref part="PWN_BTN_LED" gate="A" pin="4"/>
+<wire x1="104.14" y1="58.42" x2="99.06" y2="58.42" width="0.1524" layer="91"/>
+</segment>
 </net>
 <net name="+3V3" class="0">
-<segment>
-<pinref part="PWR_IN" gate="A" pin="2"/>
-<pinref part="+3V1" gate="G$1" pin="+3V3"/>
-</segment>
 <segment>
 <pinref part="R1" gate="G$1" pin="2"/>
@@
 </segment>
 <segment>
-<pinref part="PWR_BTN_LED" gate="1" pin="3"/>
 <pinref part="+3V6" gate="G$1" pin="+3V3"/>
-<wire x1="99.06" y1="53.34" x2="101.6" y2="53.34" width="0.1524" layer="91"/>
+<wire x1="99.06" y1="53.34" x2="104.14" y2="53.34" width="0.1524" layer="91"/>
+<pinref part="PWN_BTN_LED" gate="A" pin="2"/>
+</segment>
+<segment>
+<pinref part="PWR_CON" gate="G$1" pin="1"/>
+<pinref part="+3V1" gate="G$1" pin="+3V3"/>
+<wire x1="50.8" y1="83.82" x2="43.18" y2="83.82" width="0.1524" layer="91"/>
 </segment>
 </net>
@@
 </segment>
 <segment>
-<pinref part="ENCODER" gate="1" pin="4"/>
-<wire x1="101.6" y1="71.12" x2="93.98" y2="71.12" width="0.1524" layer="91"/>
+<wire x1="104.14" y1="71.12" x2="93.98" y2="71.12" width="0.1524" layer="91"/>
 <label x="93.98" y="71.12" size="1.27" layer="95" rot="R180" xref="yes"/>
+<pinref part="ENCODER" gate="A" pin="1"/>
 </segment>
 </net>
@@
 </segment>
 <segment>
-<pinref part="ENCODER" gate="1" pin="3"/>
-<wire x1="101.6" y1="73.66" x2="93.98" y2="73.66" width="0.1524" layer="91"/>
+<wire x1="104.14" y1="73.66" x2="93.98" y2="73.66" width="0.1524" layer="91"/>
 <label x="93.98" y="73.66" size="1.27" layer="95" rot="R180" xref="yes"/>
+<pinref part="ENCODER" gate="A" pin="2"/>
 </segment>
 </net>
@@
 </segment>
 <segment>
-<pinref part="PWR_BTN_LED" gate="1" pin="2"/>
-<wire x1="101.6" y1="55.88" x2="93.98" y2="55.88" width="0.1524" layer="91"/>
+<wire x1="104.14" y1="55.88" x2="93.98" y2="55.88" width="0.1524" layer="91"/>
 <label x="93.98" y="55.88" size="1.27" layer="95" rot="R180" xref="yes"/>
+<pinref part="PWN_BTN_LED" gate="A" pin="3"/>
 </segment>
 </net>
@@
 </segment>
 <segment>
-<pinref part="ENCODER" gate="1" pin="2"/>
-<wire x1="101.6" y1="76.2" x2="93.98" y2="76.2" width="0.1524" layer="91"/>
+<wire x1="104.14" y1="76.2" x2="93.98" y2="76.2" width="0.1524" layer="91"/>
 <label x="93.98" y="76.2" size="1.27" layer="95" rot="R180" xref="yes"/>
+<pinref part="ENCODER" gate="A" pin="3"/>
 </segment>
 </net>
@@
 </segment>
 <segment>
-<pinref part="PWR_BTN_LED" gate="1" pin="4"/>
-<wire x1="101.6" y1="50.8" x2="93.98" y2="50.8" width="0.1524" layer="91"/>
+<wire x1="104.14" y1="50.8" x2="93.98" y2="50.8" width="0.1524" layer="91"/>
 <label x="93.98" y="50.8" size="1.27" layer="95" rot="R180" xref="yes"/>
-</segment>
-</net>
+<pinref part="PWN_BTN_LED" gate="A" pin="1"/>
+</segment>
+</net>

Commit message: add missing values
Parts:
- T1: value (none) -> BC847C
Changed lines of the file:
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@@
 <part name="GND5" library="supply1" deviceset="GND" device=""/>
 <part name="+3V6" library="supply1" deviceset="+3V3" device=""/>
-<part name="T1" library="transistor" deviceset="*-NPN-" device="SOT23-BEC" technology="BC847A"/>
+<part name="T1" library="transistor" deviceset="*-NPN-" device="SOT23-BEC" technology="BC847A" value="BC847C"/>
 <part name="GND6" library="supply1" deviceset="GND" device=""/>
 <part name="R5" library="rcl" deviceset="R-EU_" device="R0805" value="10k"/>
